File: Main/mainBoard.sch (EAGLE design)
At the start: 23 parts, among them X2 JST-XH-06-PIN-LONG-PAD

Commit message: 回路図と部品配置を検討し始めた
これからも検討に検討を重ね検討したいと思う。
Parts:
- removed KICK: (no value), jst-xh:S4B-XH-A
- removed LED1, LED2, PILOT: LED-SMD, Custom_Designed_By_Yusei:LED-SMD
- removed MC1, MC33151: MC33151DR2G, MC33151DR2G:MC33151DR2G
- removed MCP2551: MCP2551-I/SN, MCP2551-I_SN:MCP2551-I/SN
- removed R11: 120, rcl:R-EU_R0603
- removed X2: JST-XH-06-PIN-LONG-PAD, Rembrandt Electronics - JST XH Connectors v1-0:JST-XH-06-PIN-LONG-PAD
- added C23: 0.1uF, SparkFun-Capacitors:0.1UF-0603-100V-10%
- added CAN, I2C: (no value), SparkFun-Connectors:CONN_04JST-PTH
- added CHK, CHK1: +3V3, SparkFun-Connectors:CONN_02
- added D2, D3, D4: (no value), SparkFun-LED:LED0603
- added R5: 120, rcl:R-EU_R0603
- added R6, R7: 1k, SparkFun-Resistors:1KOHM-0603-1/10W-1%
- added U$2: 1X7, headers(2mm):1X7
- added U$3: (no value), AE-BNO055:AE-BNO055-BO
- added U3: MCP2562-E/SN, MCP2562-E_SN:MCP2562-E/SN
Connections:
- net LINE_A0 renamed CN5
- net LINE_A1 renamed CN6
- net LINE_A2 renamed CN7
- net LINE_A3 renamed CN8
- net SLEEP renamed KICK1
- removed net +15V: MC1.VCC, MC33151.VCC
- removed net 5V: X2-4.S
- removed net GVDD_IN: X2-1.S
- removed net KICK: MC33151.LOGIC_I/P_A
- removed net KICK_V: KICK.2, MC33151.DRIVE_O/P_A
- removed net KICK_V2: KICK.3, MC1.DRIVE_O/P_A
- removed net LINE_A4: NUCLEO_MAIN.PC8
- removed net LINE_ANALOG: NUCLEO_MAIN.PB1
- removed net LINE_PWM: NUCLEO_MAIN.PB2
- removed net PH1: NUCLEO_MAIN.PB3
- removed net PH2: NUCLEO_MAIN.PB4
- removed net PH3: NUCLEO_MAIN.PB5
- removed net PH4: NUCLEO_MAIN.PB6
- removed net PVDD: X2-2.S
- removed net RASP_RX: RASP.3
- removed net RASP_TX: RASP.4
- removed net RGB_B: NUCLEO_MAIN.PA12
- removed net RGB_G: NUCLEO_MAIN.PA8
- removed net RGB_R: NUCLEO_MAIN.PC9
- removed net TR_IN: KICK.4
- removed net VSS: C2.2, C34.2, C8.2, C9.2, D1.A, NUCLEO_MAIN.VREF-, NUCLEO_MAIN.VSS, NUCLEO_MAIN.VSS1, NUCLEO_MAIN.VSS2, NUCLEO_MAIN.VSS3, PILOT.C, R2.2, R3.1, R4.2, SP.2
- new net 3V3: U$2.2, U$3.VIN
- new net BAT: NUCLEO_MAIN.PA4
- new net PHOTO: NUCLEO_MAIN.PA5
- new net USBRX: U$2.7
- new net VDD: BEAD.2, C34.1, C9.1, CAN.1, I2C.1, NUCLEO_MAIN.VBAT, NUCLEO_MAIN.VDD, NUCLEO_MAIN.VDD1, NUCLEO_MAIN.VDD2, NUCLEO_MAIN.VDD3, R1.2, R6.2, R7.2, U3.VIO
- net +5V: now also C23.1, U3.VDD; no longer KICK.1, MCP2551.VDD
- net BUZZER: now also NUCLEO_MAIN.PB2; no longer NUCLEO_MAIN.PA11
- net CANH: now also CAN.4, R5.1, U3.CANH; no longer MCP2551.CANH, X2-5.S
- net CANL: now also CAN.3, R5.2, U3.CANL; no longer MCP2551.CANL, X2-6.S
- net CANRX: now also NUCLEO_MAIN.PA11, U3.RXD; no longer MCP2551.RXD, R11.2
- net CANTX: now also NUCLEO_MAIN.PA12, U3.TXD; no longer MCP2551.TXD, R11.1
- net GND: now also C2.2, C23.2, C34.2, C8.2, C9.2, CAN.2, CHK.2, D1.A, D2.C, I2C.2, NUCLEO_MAIN.VREF-, NUCLEO_MAIN.VSS, NUCLEO_MAIN.VSS1, NUCLEO_MAIN.VSS2, NUCLEO_MAIN.VSS3, R2.2, R3.1, R4.2, SP.2, U$2.1, U$3.GND, U3.STBY, U3.VSS; no longer MC1.GND, MC33151.GND, MCP2551.RS, MCP2551.VSS, X2-3.S
- net KICK2: now also NUCLEO_MAIN.PB6; no longer MC1.LOGIC_I/P_A
- net LED1: now also D3.A; no longer LED1.A
- net LED2: now also D4.A; no longer LED2.A
- net N$1: now also D4.C; no longer LED2.C
- net N$2: now also D3.C; no longer LED1.C
- net NRST: now also U$2.5
- net POWERLED_RESISTOR: now also D2.A; no longer PILOT.A
- net SCL: now also CHK1.1, I2C.3, R6.1, U$3.SCL
- net SDA: now also CHK1.2, I2C.4, R7.1, U$3.SDA
- net SERIAL1RX: now also RASP.3
- net SERIAL1TX: now also RASP.4
- net SWCLK: now also U$2.3
- net SWDIO: now also U$2.4
- net USBTX: now also U$2.6
- net VCC: now also CHK.1; no longer BEAD.2, C34.1, C9.1, NUCLEO_MAIN.VBAT, NUCLEO_MAIN.VDD, NUCLEO_MAIN.VDD1, NUCLEO_MAIN.VDD2, NUCLEO_MAIN.VDD3, R1.2
Other:
- note removed: "Kick"
- note removed: "Motor"
- note removed: "重要"

Commit message: some update 部品配置
# ==== Emojis ====
# ✨ :sparkles: Add new feature
# ✅  :white_check_mark: Update existing feature (not bug)
# ⚠️  :warning: Fix bug/error
# 🔥  :fire: Remove files or features
# ✏️ :pencil2: Fix typos
# 📝  :memo: Update documentation
# ♻️  :recycle: Dependencies update
# 🐧  :penguin: Improved the Linux
# 🍎  :apple: Improved the macOS
# 🔖 :bookmark: Add new library
# 🎉  :tada: Initial commit

# ==== Format ====
# :emoji: Subject
#
# Commit body...

# ==== Messages ====
# 新規(ファイル)機能追加: Add
# 機能修正、既存機能追加（バグではない): Update
# リファクタリング: Clean
# ファイル名変更:
# 削除など: Remove
# バグ修正: Fix
# バージョンアップ: Upgrade
Parts:
- added JP1, JP2: (no value), adafruit:PINHD-1X6
- added Q1: BSS138, BSS138:BSS138
- CAN, I2C: device SparkFun-Connectors:CONN_04JST-PTH -> jst-xh:S4B-XH-A
Connections:
- removed net SP: D1.C, R9.2, SP.1
- new net +15V: JP2.1
- new net GPIO0: JP1.6, NUCLEO_MAIN.PA6
- new net N$3: D1.C, SP.1
- new net N$4: D1.A, Q1.D, SP.2
- net +5V: now also JP2.2
- net BAT: now also JP1.1
- net BUZZER: now also Q1.G
- net CANH: now also CAN.1, JP1.2; no longer CAN.4
- net CANL: now also CAN.2, JP1.3; no longer CAN.3
- net DRIB_PWM: now also JP1.4
- net GND: now also CAN.3, I2C.3, JP2.4, Q1.S, R9.2; no longer CAN.2, D1.A, I2C.2, SP.2
- net KICK1: now also JP2.5
- net KICK2: now also JP2.6
- net PHOTO: now also JP1.5
- net SCL: now also I2C.2; no longer I2C.3
- net SDA: now also I2C.1; no longer I2C.4
- net VDD: now also CAN.4, I2C.4, JP2.3; no longer CAN.1, I2C.1
Other:
- note removed: "Recommended"
- moved on the sheet: CAN, D1, I2C, R9, SP

Commit message: POWERをした
Connections:
- removed net VCC: CHK.1
- net VDD: now also CHK.1
Changed lines of the file:
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@@
 <class number="0" name="default" width="0.3" drill="0">
 </class>
-<class number="1" name="New" width="0.7" drill="0">
-<clearance class="1" value="0.2032"/>
+<class number="1" name="New" width="0.3" drill="0">
 </class>
-<class number="2" name="n" width="0.7" drill="0">
-<clearance class="2" value="0.2032"/>
+<class number="2" name="n" width="0.3" drill="0">
 </class>
 </classes>
@@
 <pinref part="CAN" gate="G$1" pin="4"/>
 </segment>
-</net>
-<net name="3V3" class="0">
-<segment>
-<pinref part="U$3" gate="G$1" pin="VIN"/>
-<wire x1="208.28" y1="127" x2="208.28" y2="121.92" width="0.1524" layer="91"/>
-<label x="208.28" y="121.92" size="0.762" layer="95" rot="R270" xref="yes"/>
-</segment>
-<segment>
-<pinref part="U$2" gate="G$1" pin="2"/>
-<wire x1="22.86" y1="7.62" x2="20.32" y2="7.62" width="0.1524" layer="91"/>
-<label x="20.32" y="7.62" size="0.762" layer="95" rot="R180" xref="yes"/>
-</segment>
-</net>
-<net name="USBRX" class="0">
-<segment>
-<pinref part="U$2" gate="G$1" pin="7"/>
-<wire x1="22.86" y1="20.32" x2="20.32" y2="20.32" width="0.1524" layer="91"/>
-<label x="20.32" y="20.32" size="0.762" layer="95" rot="R180" xref="yes"/>
-</segment>
-</net>
-<net name="BAT" class="0">
-<segment>
-<wire x1="71.12" y1="132.08" x2="58.42" y2="132.08" width="0.1524" layer="91"/>
-<label x="58.42" y="132.08" size="0.762" layer="95" rot="R180" xref="yes"/>
-<pinref part="JP1" gate="A" pin="1"/>
-</segment>
-<segment>
-<wire x1="60.96" y1="20.32" x2="60.96" y2="12.7" width="0.1524" layer="91"/>
-<label x="60.96" y="12.7" size="0.762" layer="95" rot="R270" xref="yes"/>
-<pinref part="NUCLEO_MAIN" gate="G$1" pin="PA4"/>
-</segment>
-</net>
-<net name="KICK1" class="0">
-<segment>
-<pinref part="NUCLEO_MAIN" gate="G$1" pin="PB7"/>
-<wire x1="66.04" y1="83.82" x2="66.04" y2="91.44" width="0.1524" layer="91"/>
-<label x="66.04" y="91.44" size="0.762" layer="95" rot="R90" xref="yes"/>
-</segment>
-<segment>
-<wire x1="40.64" y1="121.92" x2="27.94" y2="121.92" width="0.1524" layer="91"/>
-<label x="27.94" y="121.92" size="0.762" layer="95" rot="R180" xref="yes"/>
-<pinref part="JP2" gate="A" pin="5"/>
-</segment>
-</net>
-<net name="VCC" class="0">
 <segment>
 <pinref part="CHK" gate="G$1" pin="1"/>
@@
 </segment>
 </net>
+<net name="3V3" class="0">
+<segment>
+<pinref part="U$3" gate="G$1" pin="VIN"/>
+<wire x1="208.28" y1="127" x2="208.28" y2="121.92" width="0.1524" layer="91"/>
+<label x="208.28" y="121.92" size="0.762" layer="95" rot="R270" xref="yes"/>
+</segment>
+<segment>
+<pinref part="U$2" gate="G$1" pin="2"/>
+<wire x1="22.86" y1="7.62" x2="20.32" y2="7.62" width="0.1524" layer="91"/>
+<label x="20.32" y="7.62" size="0.762" layer="95" rot="R180" xref="yes"/>
+</segment>
+</net>
+<net name="USBRX" class="0">
+<segment>
+<pinref part="U$2" gate="G$1" pin="7"/>
+<wire x1="22.86" y1="20.32" x2="20.32" y2="20.32" width="0.1524" layer="91"/>
+<label x="20.32" y="20.32" size="0.762" layer="95" rot="R180" xref="yes"/>
+</segment>
+</net>
+<net name="BAT" class="0">
+<segment>
+<wire x1="71.12" y1="132.08" x2="58.42" y2="132.08" width="0.1524" layer="91"/>
+<label x="58.42" y="132.08" size="0.762" layer="95" rot="R180" xref="yes"/>
+<pinref part="JP1" gate="A" pin="1"/>
+</segment>
+<segment>
+<wire x1="60.96" y1="20.32" x2="60.96" y2="12.7" width="0.1524" layer="91"/>
+<label x="60.96" y="12.7" size="0.762" layer="95" rot="R270" xref="yes"/>
+<pinref part="NUCLEO_MAIN" gate="G$1" pin="PA4"/>
+</segment>
+</net>
+<net name="KICK1" class="0">
+<segment>
+<pinref part="NUCLEO_MAIN" gate="G$1" pin="PB7"/>
+<wire x1="66.04" y1="83.82" x2="66.04" y2="91.44" width="0.1524" layer="91"/>
+<label x="66.04" y="91.44" size="0.762" layer="95" rot="R90" xref="yes"/>
+</segment>
+<segment>
+<wire x1="40.64" y1="121.92" x2="27.94" y2="121.92" width="0.1524" layer="91"/>
+<label x="27.94" y="121.92" size="0.762" layer="95" rot="R180" xref="yes"/>
+<pinref part="JP2" gate="A" pin="5"/>
+</segment>
+</net>
