File: Power/powerBoad.brd (EAGLE design)
At the start: 67 x 59.7 mm, 34 parts, among them CON1 MR30PW-M, CON2 XT30PW-M, CON3 XT30PW-M, U1 V7805-1000, U2 LD1117S33CTR, U3 MC33151DR2G, U4 MC33151DR2G

Commit message: some fix
Routing:
- net N$2: track 2.22 -> 0.00 mm
- net N$3: track 1.91 -> 0.00 mm
Changed lines of the file:
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@@
 <wire x1="2.54" y1="37.94125" x2="2.54" y2="25.55875" width="0.1" layer="42"/>
 <wire x1="2.54" y1="25.55875" x2="0.3175" y2="25.55875" width="0.1" layer="42"/>
+<wire x1="-0.3175" y1="37.7825" x2="2.38125" y2="37.7825" width="0.4" layer="42"/>
 </plain>
 <attributes>
@@
 <via x="57.445" y="25.24125" extent="1-16" drill="0.6"/>
 <via x="57.445" y="30.63875" extent="1-16" drill="0.6"/>
-<via x="53.47625" y="30.63875" extent="1-16" drill="0.6"/>
-<via x="53.47625" y="25.55875" extent="1-16" drill="0.6"/>
+<via x="53.79375" y="30.63875" extent="1-16" drill="0.6"/>
+<via x="53.79375" y="25.55875" extent="1-16" drill="0.6"/>
 <via x="55.54" y="22.225" extent="1-16" drill="0.6"/>
-<via x="53.3175" y="32.86125" extent="1-16" drill="0.6"/>
+<via x="53.79375" y="32.86125" extent="1-16" drill="0.6"/>
 <via x="57.60375" y="32.86125" extent="1-16" drill="0.6"/>
-<via x="53.3175" y="34.76625" extent="1-16" drill="0.6"/>
+<via x="53.635" y="34.76625" extent="1-16" drill="0.6"/>
 <via x="56.96875" y="38.57625" extent="1-16" drill="0.6"/>
-<via x="50.93625" y="43.18" extent="1-16" drill="0.6"/>
+<via x="51.095" y="43.33875" extent="1-16" drill="0.6"/>
 <via x="15.875" y="14.9225" extent="1-16" drill="0.5"/>
 <via x="15.875" y="11.43" extent="1-16" drill="0.5"/>
@@
 <via x="18.25625" y="18.415" extent="1-16" drill="0.6"/>
 <via x="55.2225" y="40.48125" extent="1-16" drill="0.6"/>
-<via x="53.3175" y="38.735" extent="1-16" drill="0.6"/>
+<via x="53.79375" y="38.735" extent="1-16" drill="0.6"/>
 <via x="37.465" y="41.275" extent="1-16" drill="0.5"/>
 <via x="35.56" y="43.18" extent="1-16" drill="0.5"/>
@@
 <contactref element="JP2" pad="6"/>
 <wire x1="20.4655" y1="45.4025" x2="20.6375" y2="45.4025" width="0.35" layer="1"/>
-<via x="8.5725" y="34.925" extent="1-16" drill="0.5"/>
+<via x="8.5725" y="35.2425" extent="1-16" drill="0.5"/>
 <via x="21.9075" y="45.4025" extent="1-16" drill="0.5"/>
-<wire x1="15.03515" y1="41.2289" x2="8.73125" y2="34.925" width="0.35" layer="16"/>
-<wire x1="8.5725" y1="34.925" x2="8.73125" y2="34.925" width="0.35" layer="16"/>
+<wire x1="14.5589" y1="41.2289" x2="8.5725" y2="35.2425" width="0.35" layer="16"/>
 <wire x1="28.3786" y1="44.6464" x2="32.05111875" y2="44.6464" width="0.35" layer="16"/>
 <wire x1="28.3786" y1="44.6464" x2="27.6225" y2="45.4025" width="0.35" layer="16"/>
@@
 <wire x1="21.9075" y1="45.4025" x2="21.5" y2="45.4025" width="0.35" layer="1"/>
 <wire x1="21.5" y1="45.4025" x2="21.2725" y2="45.4025" width="0.35" layer="1"/>
-<wire x1="1.27" y1="36.83" x2="3.175" y2="34.925" width="0.7" layer="1"/>
-<wire x1="8.5725" y1="34.925" x2="3.175" y2="34.925" width="0.7" layer="1"/>
+<wire x1="1.27" y1="36.83" x2="3.01625" y2="35.08375" width="0.7" layer="1"/>
+<wire x1="8.5725" y1="35.2425" x2="8.41375" y2="35.08375" width="0.7" layer="1"/>
+<wire x1="8.41375" y1="35.08375" x2="3.01625" y2="35.08375" width="0.7" layer="1"/>
 <wire x1="21.5" y1="45.5" x2="20.5" y2="45.5" width="0.35" layer="1"/>
 <wire x1="20.5" y1="45.5" x2="20.4655" y2="45.4025" width="0.35" layer="1"/>
 <wire x1="21.5" y1="45.5" x2="21.5" y2="45.4025" width="0.35" layer="1"/>
-<wire x1="31.90875" y1="41.2289" x2="15.03515" y2="41.2289" width="0.35" layer="16"/>
+<wire x1="31.90875" y1="41.2289" x2="14.5589" y2="41.2289" width="0.35" layer="16"/>
 <wire x1="32.89145" y1="42.2116" x2="31.90875" y2="41.2289" width="0.35" layer="16"/>
 <wire x1="32.89145" y1="43.80606875" x2="32.89145" y2="42.2116" width="0.35" layer="16"/>
@@
 <wire x1="28.56175" y1="45.56125" x2="28.403" y2="45.4025" width="0.5" layer="1"/>
 <via x="8.5725" y="33.655" extent="1-16" drill="0.5"/>
-<wire x1="15.5575" y1="40.64" x2="8.5725" y2="33.655" width="0.35" layer="16"/>
-<wire x1="15.5575" y1="40.64" x2="32.22625" y2="40.64" width="0.35" layer="16"/>
+<wire x1="15.08125" y1="40.64" x2="8.5725" y2="34.13125" width="0.35" layer="16"/>
+<wire x1="8.5725" y1="34.13125" x2="8.5725" y2="33.655" width="0.35" layer="16"/>
+<wire x1="15.08125" y1="40.64" x2="32.22625" y2="40.64" width="0.35" layer="16"/>
 <wire x1="33.6088125" y1="42.0225625" x2="32.22625" y2="40.64" width="0.35" layer="16"/>
 <wire x1="33.6088125" y1="44.0863125" x2="32.133875" y2="45.56125" width="0.35" layer="16"/>
@@
 <wire x1="46.4125" y1="23.6525" x2="47.14875" y2="22.91625" width="0.35" layer="1"/>
 </signal>
-<signal name="N$2">
-<wire x1="64.77" y1="37.62375" x2="66.9925" y2="37.62375" width="0.1" layer="16"/>
-</signal>
-<signal name="N$3">
-<wire x1="0.635" y1="37.94125" x2="2.54" y2="37.94125" width="0.1" layer="16"/>
-</signal>
 </signals>
