File: 2024/PhotoSensorBoard/PhotoSensorBoard/PhotoSensorBoard.kicad_pcb (KiCad board)
At the start: 2 copper layers, 3 parts, among them J1 Conn_01x02_Pin

Commit message: ✨Production!!
Parts:
- added D3: LED, LED_THT:LED_D3.0mm, F.Cu at (37.0, 0.73)
- added D4: LED, LED_THT:LED_D3.0mm, F.Cu at (25.0, 0.73)
- added J2: Conn_01x02_Pin, Resistor_SMD:R_0815_2038Metric_Pad1.20x4.05mm_HandSolder, F.Cu at (10.0, -4.00)
- added J3: Conn_01x02_Pin, Resistor_SMD:R_0815_2038Metric_Pad1.20x4.05mm_HandSolder, F.Cu at (34.0, -4.00)
- added J4: Conn_01x02_Pin, Resistor_SMD:R_0815_2038Metric_Pad1.20x4.05mm_HandSolder, F.Cu at (22.0, -4.00)
- added J5: Conn_01x02_Pin, Resistor_SMD:R_0815_2038Metric_Pad1.20x4.05mm_HandSolder, B.Cu at (-2.00, -4.00)
- added J6: Conn_01x02_Pin, Resistor_SMD:R_0815_2038Metric_Pad1.20x4.05mm_HandSolder, B.Cu at (10.0, -4.00)
- added J7: Conn_01x02_Pin, Resistor_SMD:R_0815_2038Metric_Pad1.20x4.05mm_HandSolder, B.Cu at (34.0, -4.00)
- added J8: Conn_01x02_Pin, Resistor_SMD:R_0815_2038Metric_Pad1.20x4.05mm_HandSolder, B.Cu at (22.0, -4.00)
- moved J1 127.5 mm to (-2.00, -4.00)
- moved D1 124.4 mm to (1.00, 0.73)
- moved D2 117.7 mm to (13.0, 0.73)
Connections:
- D2 pad 1: Net-(D1-K) -> Net-(D2-K)
- D2 pad 2: Net-(D1-A) -> Net-(D2-A)
Routing:
- net Net-(D4-K): track 0.00 -> 16.4 mm
- net Net-(D3-K): track 0.00 -> 16.4 mm
- net Net-(D2-K): track 0.00 -> 16.4 mm
- net Net-(D4-A): track 0.00 -> 15.0 mm
- net Net-(D3-A): track 0.00 -> 15.0 mm
- net Net-(D2-A): track 0.00 -> 15.0 mm
- net Net-(D1-K): track 7.20 -> 16.4 mm
- net Net-(D1-A): track 7.17 -> 15.0 mm
Other:
- board outline added: 46 x 20 mm
