File: 2024/KickerBoard/lt3750_0320/lt3750_0320.kicad_sch (KiCad schematic)
At the start: 37 parts, among them J1 Conn_01x12_Socket, J2 Conn_01x02_Socket, J4 Conn_01x04_Socket, J5 Conn_01x04_Socket, Q1 tk20a60u

Commit message: add Kick&Sub
Parts:
- removed D3: LED, LED_SMD:LED_0603_1608Metric, symbol Device:LED
- removed J4, J5: Conn_01x04_Socket, Connector_PinHeader_2.54mm:PinHeader_2x02_P2.54mm_Vertical, symbol Connector:Conn_01x04_Socket
- removed R8, R9: 1k, Resistor_SMD:R_0603_1608Metric, symbol Device:R
- removed TP1, TP2, TP3, TP4, TP5, TP6, TP7, TP8: TestPoint_Probe, Connector_Pin:Pin_D0.7mm_L6.5mm_W1.8mm_FlatFork, symbol Connector:TestPoint_Probe
- added C1: 1, C_0603_1608Metric, symbol Device:C
- added C10, C2, C3, C9: 0.1u, C_0603_1608Metric, symbol Device:C
- added C17, C18: 1u, C_0603_1608Metric, symbol Device:C
- added D1, D3 (x2), D5: LED, LED_SMD:LED_0603_1608Metric, symbol Device:LED
- added F2: Fuse, Fuse_0603_1608Metric, symbol Device:Fuse
- added FB1: ~, L_0603_1608Metric, symbol Device:FerriteBead
- added J3, J4: Conn_01x02_Socket, Connector_PinHeader_2.54mm:PinHeader_1x02_P2.54mm_Vertical, symbol Connector:Conn_01x02_Socket
- added J5: Conn_01x03_Female, Connector_JST:JST_XH_B3B-XH-A_1x03_P2.50mm_Vertical, symbol Connector:Conn_01x03_Female
- added R1, R5: 10k, R_0603_1608Metric, symbol Device:R
- added R2, R3, R4 (x2), R6: 1k, R_0603_1608Metric, symbol Device:R
- added U1: STM32F303K8Tx, Package_QFP:LQFP-32_7x7mm_P0.8mm, symbol MCU_ST_STM32F3:STM32F303K8Tx
- added U3: AP2112K-3.3, newinov:SOT25, symbol DCDC:AP2112K-3.3
- added U4: MAX3051, digikey-footprints:SOIC-8_W3.9mm, symbol Interface_UART:MAX3051
- R7: value 20k -> 120; footprint Resistor_SMD:R_0603_1608Metric -> R_0603_1608Metric
Connections:
- net +15V: now also J1.11 (Pin_11), J1.12 (Pin_12), R5.1; no longer J1.7 (Pin_7), J1.8 (Pin_8), R7.2
- net CHARGE: now also R4.1, U1.26 (PB3); no longer J1.5 (Pin_5)
- net CHIP: now also U1.18 (PA8); no longer J1.11 (Pin_11)
- net GND: now also J5.3 (Pin_3); no longer C1.1, C2.2, C4.2, C5.1, C6.1, C7.1, C8.1, C9.2, D2.1 (K), D4.1 (K), J1.1 (Pin_1), J1.2 (Pin_2), J1.3 (Pin_3), J1.4 (Pin_4), LT1.5 (gnd), R10.1, R3.2, R6.1, U1.10 (10OUT)
- net STRAIGHT: now also U1.13 (PA7); no longer J1.12 (Pin_12)
- net VOUT: now also J3.1 (Pin_1), J3.2 (Pin_2)
- net at D2.2 (A): now also R3.2; no longer R7.1
- net at D4.2 (A): now also R5.2
- net +5V: no longer names the net of C9.1, LT1.4 (vcc)
- net +5V: no longer J1.6 (Pin_6), R2.1
- new net: C18.1, F2.2, U3.5 (VOUT)
- new net: C3.2, U1.4 (NRST)
- new net: D3.2 (A), R4.2 (x2)
- new net: D5.2 (A), R6.2
- new net: C1.1, C2.1, FB1.2, U1.5 (VDDA)
- new net: D1.2 (A), R2.2
- new net +3.3VP: C10.1, C9.1, F2.1, FB1.1, R2.1, R6.1, U1.1 (VDD), U1.17 (VDD), U4.3 (VDD), U4.5 (SHDN)
- new net +5VP: C17.1, J1.6 (Pin_6), U3.1 (VIN), U3.3 (EN)
- new net BOOT0: R1.1, U1.27 (PB4), U1.31 (BOOT0)
- new net CANH_: J1.8 (Pin_8), R7.1, U4.7 (CANH)
- new net CANL_: J1.7 (Pin_7), R7.2, U4.6 (CANL)
- new net CAN_LED: R2.1, U1.14 (PB0)
- new net CAN_RX: U1.21 (PA11), U4.4 (RXD)
- new net CAN_TX: U1.22 (PA12), U4.1 (TXD)
- new net DEBUG_LED: R3.1, U1.15 (PB1)
- new net DONE: R4.1, U1.28 (PB5)
- new net DRI_SIGNAL: J1.5 (Pin_5), U1.29 (PB6)
- new net GNDPWR: C1.1, C1.2, C10.2, C17.2, C18.2, C2.2, C2.2, C3.1, C4.2, C5.1, C6.1, C7.1, C8.1, C9.2, C9.2, D1.1 (K), D2.1 (K), D3.1 (K), D3.1 (K), D4.1 (K), D5.1 (K), J1.1 (Pin_1), J1.2 (Pin_2), J1.3 (Pin_3), J1.4 (Pin_4), J4.1 (Pin_1), J4.2 (Pin_2), LT1.5 (gnd), R1.2, R10.1, R3.2, R6.1, U1.10 (10OUT), U1.16 (VSS), U1.32 (VSS), U3.2 (GND), U4.2 (GND), U4.8 (RS)
- new net SWCLK: J5.2 (Pin_2), U1.24 (PA14)
- new net SWDIO: J5.1 (Pin_1), U1.23 (PA13)
- new net USART1_RX: U1.20 (PA10)
- new net USART1_TX: U1.19 (PA9)

Commit message: add Kick&Sub
Parts:
- removed D3: LED, LED_SMD:LED_0603_1608Metric, symbol Device:LED
- removed J1: Conn_01x12_Socket, Connector_PinHeader_2.54mm:PinHeader_2x06_P2.54mm_Vertical, symbol Connector:Conn_01x12_Socket
- removed R4: 1k, R_0603_1608Metric, symbol Device:R
- removed R7: 120, R_0603_1608Metric, symbol Device:R
- added J6: Conn_01x14_Socket, Connector_PinHeader_2.54mm:PinHeader_2x07_P2.54mm_Vertical, symbol Connector:Conn_01x14_Socket
Connections:
- net GND is gone; now on net SWDIO: J5.3 (Pin_3)
- net +15V: now also J6.1 (Pin_1), J6.2 (Pin_2), J6.3 (Pin_3), J6.4 (Pin_4)
- net +3.3VP: now also J6.8 (Pin_8)
- net +5VP: now also J6.6 (Pin_6)
- net CAN_LED: now also U1.25 (PA15); no longer U1.14 (PB0)
- net CHARGE: now also U1.30 (PB7); no longer U1.26 (PB3)
- net CHIP: now also U1.10 (PA4); no longer U1.18 (PA8)
- net DEBUG_LED: now also U1.26 (PB3); no longer U1.15 (PB1)
- net DRI_SIGNAL: now also U1.14 (PB0), J6.5 (Pin_5); no longer U1.29 (PB6)
- net GNDPWR: now also J5.1 (Pin_1), J6.11 (Pin_11), J6.12 (Pin_12), J6.13 (Pin_13), J6.14 (Pin_14)
- net STRAIGHT: now also U1.9 (PA3); no longer U1.13 (PA7)
- net SWDIO: no longer J5.1 (Pin_1)
- net CANH_ renamed CANH
- net CANH: now also J6.9 (Pin_9)
- net CANL_ renamed CANL
- net CANL: now also J6.10 (Pin_10)
- net DONE: no longer names the net of U1.28 (PB5)
- new net TR_SIGNAL: J6.7 (Pin_7), U1.15 (PB1)
Other:
- moved on the sheet: C1, C2, FB1

Commit message: add Kick&Sub2
Connections:
- net +15V: now also C9.1, LT1.4 (vcc)
Changed lines of the file:
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@@
   (junction (at 120.904 59.436) (diameter 0) (color 0 0 0 0)
   )
+  (junction (at 63.754 70.866) (diameter 0) (color 0 0 0 0)
+  )
   (junction (at 131.064 81.534) (diameter 0) (color 0 0 0 0)
   )
@@
   )
   (junction (at 234.188 190.246) (diameter 0) (color 0 0 0 0)
+  )
+  (junction (at 63.754 61.214) (diameter 0) (color 0 0 0 0)
   )
   (junction (at 154.178 57.912) (diameter 0) (color 0 0 0 0)
@@
     (stroke (width 0) (type default))
   )
+  (wire (pts (xy 63.754 61.214) (xy 63.754 70.866))
+    (stroke (width 0) (type default))
+  )
   (wire (pts (xy 184.912 144.018) (xy 183.642 144.018))
     (stroke (width 0) (type default))
@@
     (stroke (width 0) (type default))
   )
+  (wire (pts (xy 63.754 61.214) (xy 72.39 61.214))
+    (stroke (width 0) (type default))
+  )
   (wire (pts (xy 83.566 50.038) (xy 83.566 52.832))
     (stroke (width 0) (type default))
@@
     (stroke (width 0) (type default))
   )
-  (wire (pts (xy 61.468 61.214) (xy 72.39 61.214))
-    (stroke (width 0) (type default))
-  )
+  (wire (pts (xy 61.468 61.214) (xy 63.754 61.214))
+    (stroke (width 0) (type default))
+  )

Commit message: improved schematic readability
Other:
- company: (none) -> Ri-one SSL
- title: (none) -> KickerBoard ver8.0
- moved on the sheet: C1, C10, C17, C18, C2, C3, C4, C5, C6, C7, C8, C9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
