File: 2024/SubBoard/SubBoardV1.0/SubBoardV1.0.kicad_pcb (KiCad board)
At the start: 2 copper layers, 75.4 x 60 mm, 18 parts, among them J1 Conn_01x02_Socket, J10 Conn_01x02_Socket, J11 Conn_01x03_Socket, J12 Conn_01x02_Socket, J13 Conn_01x02_Socket, J14 Conn_01x06_Socket, J15 Conn_01x06_Socket, J16 Conn_01x12_Socket, J2 Conn_01x02_Socket, J3 Conn_01x02_Socket, J4 Conn_01x02_Socket, J5 Conn_01x02_Socket, J6 Conn_01x02_Socket, J7 Conn_01x02_Socket, J8 Conn_01x02_Socket, J9 Conn_01x02_Socket

Commit message: add Kick&Sub
Parts:
- removed J16: Conn_01x12_Socket, Connector_PinHeader_2.54mm:PinHeader_2x06_P2.54mm_Vertical
- added J17: Conn_01x14_Socket, Connector_PinHeader_2.54mm:PinHeader_2x07_P2.54mm_Vertical, F.Cu at (-7.67, 26.7)
- added R1: 470, Resistor_SMD:R_0603_1608Metric, F.Cu at (19.4, -22.7)
- added R2: 20k, Resistor_SMD:R_0603_1608Metric, F.Cu at (-18.4, -22.6)
- C1, C2: value C -> 1500u; footprint Capacitor_SMD:CP_Elec_10x10 -> Capacitor_THT:CP_Radial_D12.5mm_P5.00mm
- moved C1 186.7 mm to (-7.00, -1.00)
- moved J9 185.1 mm to (-17.0, 4.00)
- moved J8 173.9 mm to (23.3, -5.55), turned to -55 degrees
- moved J11 170.4 mm to (-19.6, -18.3)
- moved J15 170.4 mm to (-6.25, 19.6), turned to 0 degrees
- moved J14 170.3 mm to (-6.25, 13.1), turned to 0 degrees
- moved J3 169.5 mm to (-22.5, 10.8), turned to -45 degrees
- moved J5 168.1 mm to (-29.3, 3.80)
- moved J6 167.9 mm to (-15.2, 17.8)
- moved J4 166.0 mm to (28.9, 0.37)
- moved J12 165.8 mm to (-17.4, -26.6), turned to 180 degrees
- moved J2 163.6 mm to (18.2, 16.5), turned to -135 degrees
- moved J13 163.1 mm to (19.4, -26.6), turned to 180 degrees
- moved J10 162.6 mm to (17.0, 4.00)
- moved J1 162.6 mm to (-26.7, -4.40)
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Connections:
- J11 pad 1: SIGNAL -> DRI_SIGNAL
- J12 pad 1: GND -> +5V
- J12 pad 2: SIGNAL -> TR_SIGNAL
- J13 pad 1: GND -> Net-(J13-Pin_1)
- J13 pad 2: +3.3V -> GND
- J14 pad 1: GND -> +15V
- J14 pad 2: +15V -> GND
- J14 pad 3: +3.3V -> +5V
- J14 pad 4: +5V -> +3.3V
- J15 pad 1: GND -> +15V
- J15 pad 2: +15V -> GND
- J15 pad 3: +3.3V -> +5V
- J15 pad 4: +5V -> +3.3V
Routing:
- net +5V: track 0.00 -> 145.9 mm
- net CANH: track 0.00 -> 113.2 mm
- net CANL: track 0.00 -> 110.7 mm
- net TR_SIGNAL: track 0.00 -> 83.2 mm
- net DRI_SIGNAL: track 0.00 -> 67.6 mm
- net +3.3V: track 0.00 -> 11.6 mm
- net GND: track 0.00 -> 7.64 mm
- net +15V: track 0.00 -> 3.30 mm
- net Net-(J13-Pin_1): track 0.00 -> 3.08 mm
- added copper zone on F.Cu, net +15V
- added copper zone on B.Cu, net GND

Commit message: add Kick&Sub2
Parts:
- added G***: LOGO, DCDC1_library:eye, B.Cu at (14.0, 0.00)
- added G***: LOGO, DCDC1_library:eye, B.Cu at (-14.0, 0.00)
- added G***: LOGO, DCDC1_library:kuti, B.Cu at (0.00, 17.0)
- added G***: LOGO, DCDC1_library:black, B.Cu at (2.75, -45.5)
- added REF**: FCC-Logo_7.3x6mm_SilkScreen, Symbol:FCC-Logo_7.3x6mm_SilkScreen, B.Cu at (0.00, 5.50)
- moved R1 1.17 mm to (18.5, -23.5), turned to 180 degrees
- moved J1 0.60 mm to (-26.7, -5.00)
Routing:
- net +5V: track 145.9 -> 148.0 mm
Other:
- board text added: "SubBoardVer1.0 20240411 KotaroOCHIISHI"

Commit message: improved schematic readability
Changed lines of the file:
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@@
     (fp_line (start 3.95 2.8) (end 3.95 -1.7)
       (stroke (width 0.1) (type solid)) (layer "F.Fab"))
-    (pad "1" thru_hole roundrect (at 0 0 315) (size 1.2 1.75) (drill 0.75) (layers "*.Cu" "*.Mask") (roundrect_rratio 0.208333)
+    (pad "1" thru_hole roundrect (at 0 0 315) (size 1.2 1.75) (drill 0.75) (layers "*.Cu" "*.Mask") (roundrect_rratio 0.2083333333)
       (net 3 "CANL") (pinfunction "Pin_1") (pintype "passive"))
     (pad "2" thru_hole oval (at 2 0 315) (size 1.2 1.75) (drill 0.75) (layers "*.Cu" "*.Mask")
@@
     (fp_line (start 14.95 0.8) (end 14.95 -3.1)
       (stroke (width 0.1) (type solid)) (layer "F.Fab"))
-    (pad "1" thru_hole roundrect (at 0 0) (size 1.7 1.85) (drill 0.85) (layers "*.Cu" "*.Mask") (roundrect_rratio 0.147059)
+    (pad "1" thru_hole roundrect (at 0 0) (size 1.7 1.85) (drill 0.85) (layers "*.Cu" "*.Mask") (roundrect_rratio 0.1470588235)
       (net 1 "+15V") (pinfunction "Pin_1") (pintype "passive"))
     (pad "2" thru_hole oval (at 2.5 0) (size 1.7 1.85) (drill 0.85) (layers "*.Cu" "*.Mask")
@@
     (fp_line (start 14.95 0.8) (end 14.95 -3.1)
       (stroke (width 0.1) (type solid)) (layer "F.Fab"))
-    (pad "1" thru_hole roundrect (at 0 0) (size 1.7 1.85) (drill 0.85) (layers "*.Cu" "*.Mask") (roundrect_rratio 0.147059)
+    (pad "1" thru_hole roundrect (at 0 0) (size 1.7 1.85) (drill 0.85) (layers "*.Cu" "*.Mask") (roundrect_rratio 0.1470588235)
       (net 1 "+15V") (pinfunction "Pin_1") (pintype "passive"))
     (pad "2" thru_hole oval (at 2.5 0) (size 1.7 1.85) (drill 0.85) (layers "*.Cu" "*.Mask")
@@
     (fp_line (start 4.95 0.8) (end 4.95 -3.1)
       (stroke (width 0.1) (type solid)) (layer "F.Fab"))
-    (pad "1" thru_hole roundrect (at 0 0 55) (size 1.7 1.85) (drill 0.85) (layers "*.Cu" "*.Mask") (roundrect_rratio 0.147059)
+    (pad "1" thru_hole roundrect (at 0 0 55) (size 1.7 1.85) (drill 0.85) (layers "*.Cu" "*.Mask") (roundrect_rratio 0.1470588235)
       (net 2 "GND") (pinfunction "Pin_1") (pintype "passive"))
     (pad "2" thru_hole oval (at 2.5 0 55) (size 1.7 1.85) (drill 0.85) (layers "*.Cu" "*.Mask")
@@
     (fp_line (start 3.95 2.8) (end 3.95 -1.7)
       (stroke (width 0.1) (type solid)) (layer "F.Fab"))
-    (pad "1" thru_hole roundrect (at 0 0 305) (size 1.2 1.75) (drill 0.75) (layers "*.Cu" "*.Mask") (roundrect_rratio 0.208333)
+    (pad "1" thru_hole roundrect (at 0 0 305) (size 1.2 1.75) (drill 0.75) (layers "*.Cu" "*.Mask") (roundrect_rratio 0.2083333333)
       (net 3 "CANL") (pinfunction "Pin_1") (pintype "passive"))
     (pad "2" thru_hole oval (at 2 0 305) (size 1.2 1.75) (drill 0.75) (layers "*.Cu" "*.Mask")
@@
     (fp_line (start 7.45 0.8) (end 7.45 -3.1)
       (stroke (width 0.1) (type solid)) (layer "F.Fab"))
-    (pad "1" thru_hole roundrect (at 0 0 270) (size 1.7 1.85) (drill 0.85) (layers "*.Cu" "*.Mask") (roundrect_rratio 0.147059)
+    (pad "1" thru_hole roundrect (at 0 0 270) (size 1.7 1.85) (drill 0.85) (layers "*.Cu" "*.Mask") (roundrect_rratio 0.1470588235)
       (net 5 "DRI_SIGNAL") (pinfunction "Pin_1") (pintype "passive"))
     (pad "2" thru_hole oval (at 2.5 0 270) (size 1.7 1.85) (drill 0.85) (layers "*.Cu" "*.Mask")
@@
     (fp_line (start 3.95 2.8) (end 3.95 -1.7)
       (stroke (width 0.1) (type solid)) (layer "F.Fab"))
-    (pad "1" thru_hole roundrect (at 0 0 55) (size 1.2 1.75) (drill 0.75) (layers "*.Cu" "*.Mask") (roundrect_rratio 0.208333)
+    (pad "1" thru_hole roundrect (at 0 0 55) (size 1.2 1.75) (drill 0.75) (layers "*.Cu" "*.Mask") (roundrect_rratio 0.2083333333)
       (net 3 "CANL") (pinfunction "Pin_1") (pintype "passive"))
     (pad "2" thru_hole oval (at 2 0 55) (size 1.2 1.75) (drill 0.75) (layers "*.Cu" "*.Mask")
@@
     (fp_line (start 4.95 0.8) (end 4.95 -3.1)
       (stroke (width 0.1) (type solid)) (layer "F.Fab"))
-    (pad "1" thru_hole roundrect (at 0 0 225) (size 1.7 1.85) (drill 0.85) (layers "*.Cu" "*.Mask") (roundrect_rratio 0.147059)
+    (pad "1" thru_hole roundrect (at 0 0 225) (size 1.7 1.85) (drill 0.85) (layers "*.Cu" "*.Mask") (roundrect_rratio 0.1470588235)
       (net 2 "GND") (pinfunction "Pin_1") (pintype "passive"))
     (pad "2" thru_hole oval (at 2.5 0 225) (size 1.7 1.85) (drill 0.85) (layers "*.Cu" "*.Mask")
@@
     (fp_line (start 4.95 0.8) (end 4.95 -3.1)
       (stroke (width 0.1) (type solid)) (layer "F.Fab"))
-    (pad "1" thru_hole roundrect (at 0 0 135) (size 1.7 1.85) (drill 0.85) (layers "*.Cu" "*.Mask") (roundrect_rratio 0.147059)
+    (pad "1" thru_hole roundrect (at 0 0 135) (size 1.7 1.85) (drill 0.85) (layers "*.Cu" "*.Mask") (roundrect_rratio 0.1470588235)
       (net 2 "GND") (pinfunction "Pin_1") (pintype "passive"))
     (pad "2" thru_hole oval (at 2.5 0 135) (size 1.7 1.85) (drill 0.85) (layers "*.Cu" "*.Mask")
@@
     (fp_line (start 3.95 2.8) (end 3.95 -1.7)
       (stroke (width 0.1) (type solid)) (layer "F.Fab"))
-    (pad "1" thru_hole roundrect (at 0 0 180) (size 1.2 1.75) (drill 0.75) (layers "*.Cu" "*.Mask") (roundrect_rratio 0.208333)
+    (pad "1" thru_hole roundrect (at 0 0 180) (size 1.2 1.75) (drill 0.75) (layers "*.Cu" "*.Mask") (roundrect_rratio 0.2083333333)
       (net 7 "+5V") (pinfunction "Pin_1") (pintype "passive"))
     (pad "2" thru_hole oval (at 2 0 180) (size 1.2 1.75) (drill 0.75) (layers "*.Cu" "*.Mask")
@@
     (fp_line (start 3.95 2.8) (end 3.95 -1.7)
       (stroke (width 0.1) (type solid)) (layer "F.Fab"))
-    (pad "1" thru_hole roundrect (at 0 0 225) (size 1.2 1.75) (drill 0.75) (layers "*.Cu" "*.Mask") (roundrect_rratio 0.208333)
+    (pad "1" thru_hole roundrect (at 0 0 225) (size 1.2 1.75) (drill 0.75) (layers "*.Cu" "*.Mask") (roundrect_rratio 0.2083333333)
       (net 3 "CANL") (pinfunction "Pin_1") (pintype "passive"))
     (pad "2" thru_hole oval (at 2 0 225) (size 1.2 1.75) (drill 0.75) (layers "*.Cu" "*.Mask")
@@
     (fp_line (start 3.95 2.8) (end 3.95 -1.7)
       (stroke (width 0.1) (type solid)) (layer "F.Fab"))
-    (pad "1" thru_hole roundrect (at 0 0 180) (size 1.2 1.75) (drill 0.75) (layers "*.Cu" "*.Mask") (roundrect_rratio 0.208333)
+    (pad "1" thru_hole roundrect (at 0 0 180) (size 1.2 1.75) (drill 0.75) (layers "*.Cu" "*.Mask") (roundrect_rratio 0.2083333333)
       (net 9 "Net-(J13-Pin_1)") (pinfunction "Pin_1") (pintype "passive"))
     (pad "2" thru_hole oval (at 2 0 180) (size 1.2 1.75) (drill 0.75) (layers "*.Cu" "*.Mask")
@@
     (fp_line (start 4.95 0.8) (end 4.95 -3.1)
       (stroke (width 0.1) (type solid)) (layer "F.Fab"))
-    (pad "1" thru_hole roundrect (at 0 0 305) (size 1.7 1.85) (drill 0.85) (layers "*.Cu" "*.Mask") (roundrect_rratio 0.147059)
+    (pad "1" thru_hole roundrect (at 0 0 305) (size 1.7 1.85) (drill 0.85) (layers "*.Cu" "*.Mask") (roundrect_rratio 0.1470588235)
       (net 2 "GND") (pinfunction "Pin_1") (pintype "passive"))
     (pad "2" thru_hole oval (at 2.5 0 305) (size 1.7 1.85) (drill 0.85) (layers "*.Cu" "*.Mask")
