File: 2024/SubUnit/SubUnit_V1/SubBoardV1.0/SubBoardV1.0.kicad_pcb (KiCad board)
At the start: 2 copper layers, 75.4 x 60 mm, 25 parts, among them J1 Conn_01x02_Socket, J10 Conn_01x02_Socket, J11 Conn_01x03_Socket, J12 Conn_01x02_Socket, J13 Conn_01x02_Socket, J14 Conn_01x06_Socket, J15 Conn_01x06_Socket, J17 Conn_01x14_Socket, J2 Conn_01x02_Socket, J3 Conn_01x02_Socket, J4 Conn_01x02_Socket, J5 Conn_01x02_Socket, J6 Conn_01x02_Socket, J7 Conn_01x02_Socket, J8 Conn_01x02_Socket, J9 Conn_01x02_Socket

Commit message: キッカー基板V2仮
Parts:
- removed the G*** at (-14.0, 0.00)
- removed the G*** at (0.00, 17.0)
- removed the G*** at (2.75, -45.5)
