File: 2024/MainBoard/MainBoard_V5.1/MainBoard/MainBoard.kicad_sch (KiCad schematic)
At the start: 110 parts, among them J1 Raspberry_Pi_2_3, J11 //ADC2, J12 //ADC2, J13 Drib, J14 UART, J15 TFT3, J16 CAN_CON, J2 fan, J3 USB_C_Receptacle_USB2.0_16P, J4 metor, J6 Debug, J7 //ADC0, J8 MOLEX MINISPOX, Q1 DMMT5401, Q2 Q_NMOS_GSD, Q4 Q_PMOS_GDS, SW1 SW_MEC_5E, SW2 Ras_1, SW3 Ras_2, SW4 SW_Wuerth_450301014042, SW5 SW_MEC_5E, U1 STM32F446RETx, U10 MPU9250, U2 CH340E, U3 MOUDLE-SEEEDUINO-XIAO, U6 BNO055, U7 AZ1117-3.3, U8 MAX3051, U9 LM39300R-5.0, Y1 CSTNE16M0V530000R0

Commit message: 修正版
Parts:
- removed U9: LM39300R-5.0, MainBoard:LM39300, symbol Regulator_Linear:AZ1117-3.3
- added U11: LM1084-5.0, Package_TO_SOT_SMD:TO-263-3_TabPin2, symbol Regulator_Linear:LM1084-5.0
- C19, C20, C21, C24: value 330u -> 1000u; footprint Capacitor_SMD:CP_Elec_8x11.9 -> Capacitor_SMD:CP_Elec_8x10.5
- C23, C25: value 330u -> 100u; footprint Capacitor_SMD:CP_Elec_8x11.9 -> Capacitor_SMD:CP_Elec_6.3x5.4_Nichicon
- C27: value 330u -> 47u; footprint Capacitor_SMD:CP_Elec_8x11.9 -> Capacitor_SMD:CP_Elec_6.3x5.4_Nichicon
Connections:
- net +5V: now also U11.2 (VO)
- net +6V: now also U11.3 (VI)
- net GND: now also U11.1 (GND); no longer C20.2
