File: 2024/SubUnit/SubUnit_V3/SubBoard_V3/SubBoard_V3.kicad_sch (KiCad schematic)
At the start: 28 parts, among them J1 Conn_01x02_Socket, J10 Conn_01x02_Socket, J11 Conn_01x03_Socket, J12 Conn_01x02_Socket, J13 Conn_01x02_Socket, J14 Conn_01x05_Socket, J15 Conn_01x05_Socket, J16 Conn_01x02_Socket, J18 Conn_01x07_Socket, J19 Conn_01x07_Socket, J2 Conn_01x02_Socket, J3 Conn_01x02_Socket, J4 Conn_01x02_Socket, J5 Conn_01x02_Socket, J6 Conn_01x02_Socket, J7 Conn_01x02_Socket, J8 Conn_01x02_Socket, J9 Conn_01x02_Socket

Commit message: 発注分
Parts:
- added R1: 200Ω, Resistor_SMD:R_0603_1608Metric, symbol Device:R
- J12, J13: footprint Connector_JST:JST_PH_S2B-PH-K_1x02_P2.00mm_Horizontal -> Connector_JST:JST_PH_B2B-PH-K_1x02_P2.00mm_Vertical
Connections:
- net +6V: now also R1.1; no longer J12.1 (Pin_1)
- new net: J12.1 (Pin_1), R1.2
Changed lines of the file:
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@@
+    (stroke (width 0) (type default))
+  )
+  (wire (pts (xy 68.834 162.306) (xy 72.644 162.306))
     (stroke (width 0) (type default))
   )
@@
     (stroke (width 0) (type default))
   )
+  (wire (pts (xy 56.642 162.306) (xy 61.214 162.306))
+    (stroke (width 0) (type default))
+  )
   (wire (pts (xy 125.73 100.33) (xy 127.762 100.33))
     (stroke (width 0) (type default))
@@
   )
   (wire (pts (xy 113.792 54.61) (xy 117.094 54.61))
-    (stroke (width 0) (type default))
-  )
-  (wire (pts (xy 72.644 162.306) (xy 56.642 162.306))
     (stroke (width 0) (type default))
   )
@@
     )
   )
+  (symbol (lib_id "Device:R") (at 65.024 162.306 270) (unit 1)
+    (in_bom yes) (on_board yes) (dnp no)
+    (property "Reference" "R1" (at 68.072 164.846 90)
+      (effects (font (size 1.27 1.27)))
+    )
+    (property "Value" "200Ω" (at 60.706 164.846 90)
+      (effects (font (size 1.27 1.27)))
+    )
+    (property "Footprint" "Resistor_SMD:R_0603_1608Metric" (at 65.024 160.528 90)
+      (effects (font (size 1.27 1.27)) hide)
+    )
+    (property "Datasheet" "~" (at 65.024 162.306 0)
+      (effects (font (size 1.27 1.27)) hide)
+    )
+    (pin "1")
+    (pin "2")
+    (instances
+      (project "lt3750_0320"
+        (path "/bbbce0f9-d085-4300-a0ee-67783cc084cd"
+          (reference "R1") (unit 1)
+        )
+      )
+      (project "SubBoard_V3"
+        (path "/f588d83c-66c1-45ba-96cd-d938f5aa02a1"
+          (reference "R5") (unit 1)
+        )
+      )
+    )
+  )
   (symbol (lib_id "power:+6V") (at 76.708 165.354 0) (unit 1)
     (in_bom yes) (on_board yes) (dnp no) (fields_autoplaced)
@@
       (effects (font (size 1.27 1.27)) hide)
     )
-    (property "Footprint" "Connector_JST:JST_PH_S2B-PH-K_1x02_P2.00mm_Horizontal" (at 51.308 172.466 0)
+    (property "Footprint" "Connector_JST:JST_PH_B2B-PH-K_1x02_P2.00mm_Vertical" (at 51.308 172.466 0)
       (effects (font (size 1.27 1.27)) hide)
     )
@@
       (effects (font (size 1.27 1.27)) hide)
     )
-    (property "Footprint" "Connector_JST:JST_PH_S2B-PH-K_1x02_P2.00mm_Horizontal" (at 51.562 162.306 0)
-      (effects (font (size 1.27 1.27)) hide)
-    )
+    (property "Footprint" "Connector_JST:JST_PH_B2B-PH-K_1x02_P2.00mm_Vertical" (at 51.562 162.306 0)
+      (effects (font (size 1.27 1.27)) hide)
+    )
