File: 2026/PCB/PowerUnit/PowerBoard/PowerBoard_V26_3_0/BoostCircuit.kicad_sch (KiCad schematic)
At the start: 49 parts, among them J6 Micro-Fit_3P, J7 Micro-Fit_3P, J8 Micro-Fit_2P, J9 Micro-Fit_2P, Q3 FDS2582, Q4 IPD50R3K0CEAUMA1, Q5 HGT1S10N120BNST, Q6 HGT1S10N120BNST, T1 750032052, U10 R-78K12-0.5, U8 LT3751UFD, U9 FAN3227TMX

Commit message: 修正、出力
Parts:
- renumbered C38 to C39, C39 to C40, C40 to C41, C41 to C42, C42 to C43, C43 to C44, C44 to C45, C45 to C46, C46 to C47, C47 to C48, C48 to C49, C49 to C50, C50 to C51, C51 to C52, R24 to R26, R25 to R27, R26 to R28, R27 to R29, R28 to R30, R29 to R31, R30 to R32, R31 to R33, R32 to R34, R33 to R35, R34 to R36, R35 to R37, R36 to R38, R37 to R39, R38 to R40, R39 to R41, R40 to R42, R41 to R43
