File: 2026/PCB/WheelUnit/WheelDriver/WheelDriver_V26_3_2/WheelDriver_V26_3_2.kicad_pcb (KiCad board)
At the start: 4 copper layers, 86 x 65 mm, 338 parts, among them J1 BLDC1, J10 PCO_GND, J11 PCO_GND, J12 PCO_50V, J13 PCO_50V, J14 MD_UART, J15 PCO_3V3, J16 PCO_3V3, J2 ENC1, J3 WRITE_CO, J4 BLDC2, J5 ENC2, J6 BLDC3, J7 ENC3, J8 BLDC4, J9 ENC4, SW1 SW_DIP_x02, SW2 SW_DIP_x02, SW3 SW_MEC_5E, SW4 SW_MEC_5E, SW5 SW_MEC_5E, SW6 SW_MEC_5E, U1 CD74HC4066PWR, U2 CD74HC4066PWR, U3 CD74HC4066PWR, U4 CD74HC4066PWR, U5 CD74HC4066PWR, U6 TMP235AQDCKRQ1, U7 TMP235AQDCKRQ1, U8 TMP235AQDCKRQ1, U9 TMP235AQDCKRQ1

Commit message: 製造ファイル出力
Other:
- board text added: "WHITE FANG 465 V26.3.2"
- board text added: "Wheel Driver Rot_No.27JAN2026-26-3-2 Git_No.7d93137f9f1dc66407c5116ae2753e106fe6112a"
- board text removed: "WHITE FANG 465 V26.3.1"
- board text removed: "Wheel Driver Rot_No.17DEC2025-26-3-1 Git_No.5e8e394a67a1cfcad7f27511a22be45c2a132782"

Commit message: 書き込み修正
Parts:
- removed R123, R124, R125, R126: 1k, Resistor_SMD:R_0603_1608Metric_Pad0.98x0.95mm_HandSolder
- removed SW1, SW2: SW_DIP_x02, WheelUnit_LIB_FTP:CFS0201TB
- removed U1, U2, U3, U4, U5: CD74HC4066PWR, Package_SO:TSSOP-14_4.4x5mm_P0.65mm
- added J17: Conn_01x05_Pin, Connector_PinHeader_2.54mm:PinHeader_1x05_P2.54mm_Vertical, F.Cu at (227.3, 118.3)
- added J18: Conn_01x05_Pin, Connector_PinHeader_2.54mm:PinHeader_1x05_P2.54mm_Vertical, F.Cu at (227.3, 115.7)
- added J19: Conn_01x05_Pin, Connector_PinHeader_2.54mm:PinHeader_1x05_P2.54mm_Vertical, F.Cu at (224.7, 115.7)
- added J20: Conn_01x05_Pin, Connector_PinHeader_2.54mm:PinHeader_1x05_P2.54mm_Vertical, F.Cu at (224.7, 118.3)
- J3: value WRITE_CO -> Conn_01x02_Pin; footprint Connector_JST:JST_PH_S7B-PH-K_1x07_P2.00mm_Horizontal -> Connector_PinHeader_2.54mm:PinHeader_1x02_P2.54mm_Vertical
- moved J3 13.6 mm to (224.7, 103.0), turned to 90 degrees
- moved D3 2.31 mm to (228.3, 92.8)
- moved D4 2.31 mm to (223.7, 92.8)
- moved R7 2.31 mm to (226.7, 92.8)
- moved R8 2.31 mm to (225.2, 92.8)
- moved C111 2.31 mm to (227.8, 100.0)
- moved C112 2.31 mm to (224.2, 100.0)
- moved D14 2.31 mm to (227.8, 95.4)
- moved D15 2.31 mm to (227.8, 96.9)
- moved D16 2.31 mm to (227.8, 98.4)
- moved D21 2.31 mm to (224.2, 98.4)
- moved D22 2.31 mm to (224.2, 96.9)
- moved D23 2.31 mm to (224.2, 95.4)
- moved G*** 1.70 mm to (221.2, 122.6)
- moved G*** 1.70 mm to (219.7, 99.5)
Connections:
- net /NRST_1 renamed /STSPIN32G4_MAC/NRST
- net /NRST_2 renamed /STSPIN32G4_MAC1/NRST
- net /NRST_3 renamed /STSPIN32G4_MAC2/NRST
- net /NRST_4 renamed /STSPIN32G4_MAC3/NRST
- J3 pad 1: /USART1_RX -> +3.3V
- J3 pad 2: /USART1_TX -> GND
Routing:
- net /USART1_RX: track 55.3 -> 0.00 mm, vias 5 -> 0
- net /WRITE_SW2: track 54.9 -> 0.00 mm, vias 4 -> 0
- net /SWDIO: track 53.0 -> 0.00 mm, vias 4 -> 0
- net /WRITE_SW3: track 47.0 -> 0.00 mm, vias 2 -> 0
- net /USART1_TX: track 46.6 -> 0.00 mm, vias 5 -> 0
- net /SWCLK: track 46.0 -> 0.00 mm, vias 4 -> 0
- net /WRITE_SW4: track 44.5 -> 0.00 mm, vias 3 -> 0
- net /NRST: track 40.1 -> 0.00 mm, vias 1 -> 0
- net /WRITE_SW1: track 39.4 -> 0.00 mm, vias 2 -> 0
- net /STSPIN32G4_MAC1/USART_RX: track 31.3 -> 0.00 mm, vias 2 -> 0
- net /STSPIN32G4_MAC1/USART_TX: track 31.0 -> 0.00 mm, vias 2 -> 0
- net /STSPIN32G4_MAC3/SWCLK: track 27.1 -> 0.00 mm, vias 2 -> 0
- net +3.3V: track 351.8 -> 324.9 mm, vias 23 -> 22
- net /STSPIN32G4_MAC2/SWCLK: track 26.7 -> 0.00 mm, vias 2 -> 0
- net /STSPIN32G4_MAC1/SWCLK: track 26.4 -> 0.00 mm, vias 2 -> 0
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Other:
- board text added: "Wheel Driver Rot_No.27JAN2026-26-4-23 Git_No.7d93137f9f1dc66407c5116ae2753e106fe6112a"
- board text removed: "NRST"
- board text removed: "SWCLK"
- board text removed: "SWDIO"
- board text removed: "TX"
- board text removed: "Wheel Driver Rot_No.27JAN2026-26-3-2 Git_No.7d93137f9f1dc66407c5116ae2753e106fe6112a"

Commit message: 修正１
Parts:
- moved J17 10.2 mm to (227.3, 128.4), turned to 180 degrees
- moved J19 10.2 mm to (224.7, 105.6), turned to 0 degrees
Routing:
- net /STSPIN32G4_MAC3/USART_RX: track 0.00 -> 27.4 mm, vias 0 -> 1
- net /STSPIN32G4_MAC3/USART_TX: track 0.00 -> 25.1 mm, vias 0 -> 2
- net /STSPIN32G4_MAC2/SWDIO: track 0.00 -> 24.5 mm, vias 0 -> 2
- net /STSPIN32G4_MAC3/SWDIO: track 0.00 -> 23.7 mm, vias 0 -> 2
- net /STSPIN32G4_MAC2/USART_TX: track 0.00 -> 22.5 mm, vias 0 -> 2
- net /STSPIN32G4_MAC2/USART_RX: track 0.00 -> 22.1 mm, vias 0 -> 1
- net /STSPIN32G4_MAC2/SWCLK: track 0.00 -> 21.9 mm, vias 0 -> 1
- net /STSPIN32G4_MAC3/SWCLK: track 0.00 -> 21.1 mm, vias 0 -> 1
- net /STSPIN32G4_MAC2/NRST: track 3.20 -> 16.9 mm, vias 0 -> 2
- net /STSPIN32G4_MAC3/NRST: track 3.20 -> 16.1 mm, vias 0 -> 2
- net +3.3V: track 324.9 -> 325.7 mm, vias 22 -> 23
- net +8V: track 205.3 -> 205.8 mm
