File: 2026/PCB/DribblerUnit/dribbler_md_V26_1_2/dribbler_md_V26_1_2.kicad_pcb (KiCad board)
At the start: 2 copper layers, 82 x 26 mm, 125 parts, among them J1 Conn_01x05_Pin, J2 Conn_01x04_Pin, J3 Conn_01x02_Pin, J4 Conn_01x04_Pin, J4 Conn_01x07_Pin, J8 Conn_01x02_Socket, SW2 SW_MEC_5E, SW4 SW_MEC_5E, U1 MAX3051, U2 STS8DN3LLH5, U3 STS8DN3LLH5, U4 DRV8701, U5 STM32F446RETx, Y1 Crystal_GND2

Commit message: 製造ファイル出力
Other:
- board text added: "Dribbler Driver V26.1.2"
- board text added: "Git_No.6b21344809c7edc349b4 b9a6935b21bcc061b37c"
- board text added: "Rot_No.17MAY2026-26-1-2"
- board text removed: "Dribbler Driver V26.1.1"
- board text removed: "Git_No.17fe4d9b004896a47c4d5 713bca41b0264ba8419"
- board text removed: "Rot_No.17DEC2025-26-1-1"
Changed lines of the file:
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@@
 		)
 	)
-	(gr_text "Dribbler Driver V26.1.1 "
+	(gr_text "Dribbler Driver V26.1.2"
 		(at 212.374767 101.493427 0)
 		(layer "B.SilkS")
@@
 			(justify left bottom mirror)
 		)
-		(render_cache "Dribbler Driver V26.1.1 " 0
+		(render_cache "Dribbler Driver V26.1.2" 0
 			(polygon
 				(pts
@@
 			(polygon
 				(pts
-					(xy 196.339662 101.289427) (xy 196.481225 101.289427) (xy 196.481225 100.351534) (xy 196.535805 100.399308)
-					(xy 196.612273 100.452138) (xy 196.69415 100.498713) (xy 196.763325 100.529734) (xy 196.763325 100.38905)
-					(xy 196.653226 100.324503) (xy 196.557221 100.247413) (xy 196.501107 100.189321) (xy 196.459884 100.135123)
-					(xy 196.431473 100.084235) (xy 196.339662 100.084235)
+					(xy 196.127403 101.153432) (xy 196.127403 101.289427) (xy 196.887706 101.289427) (xy 196.88289 101.233713)
+					(xy 196.863575 101.170716) (xy 196.826926 101.098697) (xy 196.77889 101.031504) (xy 196.703648 100.949401)
+					(xy 196.594065 100.849496) (xy 196.46361 100.731907) (xy 196.381462 100.646906) (xy 196.334875 100.587179)
+					(xy 196.299481 100.523756) (xy 196.27985 100.466649) (xy 196.273667 100.414549) (xy 196.281077 100.355149)
+					(xy 196.30211 100.305777) (xy 196.336328 100.264266) (xy 196.381694 100.231797) (xy 196.432534 100.212687)
+					(xy 196.490799 100.206161) (xy 196.55319 100.21319) (xy 196.606303 100.233585) (xy 196.652451 100.268003)
+					(xy 196.685953 100.312315) (xy 196.707597 100.370128) (xy 196.715539 100.445323) (xy 196.860864 100.431255)
+					(xy 196.846553 100.344445) (xy 196.821943 100.273964) (xy 196.788426 100.217036) (xy 196.74657 100.171429)
+					(xy 196.69402 100.133772) (xy 196.634123 100.106773) (xy 196.565445 100.090074) (xy 196.486012 100.084235)
+					(xy 196.399803 100.091216) (xy 196.328513 100.110879) (xy 196.269127 100.142368) (xy 196.219641 100.186304)
+					(xy 196.169387 100.257513) (xy 196.139451 100.334228) (xy 196.129283 100.418286) (xy 196.137039 100.493465)
+					(xy 196.160369 100.566738) (xy 196.200065 100.63913) (xy 196.252706 100.70744) (xy 196.338849 100.79951)
+					(xy 196.468744 100.921157) (xy 196.63185 101.072685) (xy 196.66571 101.113736) (xy 196.691604 101.153432)
 				)
 			)
@@
 		)
 	)
-	(gr_text "Git_No.17fe4d9b004896a47c4d5\n       713bca41b0264ba8419"
+	(gr_text "Git_No.6b21344809c7edc349b4\n       b9a6935b21bcc061b37c"
 		(at 194.09368 96.144996 0)
 		(layer "B.SilkS")
@@
 		)
 	)
-	(gr_text "Rot_No.17DEC2025-26-1-1"
+	(gr_text "Rot_No.17MAY2026-26-1-2"
 		(at 194.39848 93.554196 0)
 		(layer "B.SilkS")
