File: 2026/PCB/OtherBoards/OtherBoards_V26_2/OtherBoards_V26_2.kicad_pcb (KiCad board)
At the start: 2 copper layers, 65 x 94 mm, 76 parts, among them J1 Conn_01x03

Commit message: 修正&製造ファイル出力
Connections:
- U1 pad 5: GND -> unconnected-(U1-PGO-Pad5) (x8)
- U1 pad 6: GND -> unconnected-(U1-SDA-Pad6) (x8)
- U1 pad 7: GND -> unconnected-(U1-SCL-Pad7) (x8)
- U1 pad 8: GND -> unconnected-(U1-DIR-Pad8) (x8)
Routing:
- net GND: vias 72 -> 80
