File: 2026/PCB/MainBoard/MainBoard_V26_2_1/MainBoard_V26_2_1.kicad_pcb (KiCad board)
At the start: 2 copper layers, 100 x 65 mm, 94 parts, among them J1 Raspberry_Pi_2_3, J15 TFT3, J16 CAN_CON, J2 fan, J3 MOLEX, J5 Conn_01x05_Socket, J6 Debug, Q1 Q_NMOS_GSD, Q2 Q_NMOS_GSD, SW1 SW_MEC_5E, SW2 Ras_1, SW3 Ras_2, U1 STM32F446RETx, U2 LMR51460FSQDRRRQ1, U3 MOUDLE-SEEEDUINO-XIAO, U5 MCP1703AT-3302E/CB, U6 LSM6DSO32XTR, U7 LTC4451AV-TRPBF, U8 MAX3051, U9 LTC4451AV-TRPBF, Y1 CSTNE16M0V530000R0

Commit message: 途中保存
Parts:
- C12, C8: moved to F.Cu
- moved C8 28.2 mm to (206.4, 87.2), turned to -90 degrees
- moved C12 5.75 mm to (230.2, 121.7), turned to 180 degrees
- moved C6 1.44 mm to (237.6, 80.8)
- moved C2 1.44 mm to (236.3, 79.6)
Routing:
- net +3.3V: track 155.8 -> 224.9 mm, vias 15 -> 17
- net MOSI: track 0.00 -> 41.0 mm, vias 0 -> 2
- net MISO: track 0.00 -> 35.7 mm, vias 0 -> 1
- net SCK: track 0.00 -> 32.3 mm, vias 0 -> 2
- net LED0: track 7.54 -> 39.8 mm
- net LED1: track 12.6 -> 40.4 mm
- net UI_Audio: track 96.3 -> 123.8 mm, vias 0 -> 2
- net T_CS: track 0.00 -> 24.0 mm, vias 0 -> 1
- net LED2: track 15.9 -> 39.7 mm
- net HEART_BEAT_LED: track 18.4 -> 40.3 mm
- net LED_CS: track 0.00 -> 20.9 mm, vias 0 -> 1
- net UART4_RX: track 17.2 -> 38.0 mm
- net UART4_TX: track 16.6 -> 35.9 mm
- net Reset: track 0.00 -> 17.3 mm
- net D/C: track 0.00 -> 16.3 mm
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Other:
- board text added: "MainBoard V26.2.1"
- board text removed: "MainBoard V26.1.3"

Commit message: 修正完了。理想ダイオード変更前
Parts:
- added B5819W-TP1: D, Diode_SMD:D_SOD-123, F.Cu at (227.2, 122.4)
- added B5819W-TP2: D, Diode_SMD:D_SOD-123, F.Cu at (178.4, 73.7)
- added Q3: Q_NMOS_GSD, Package_TO_SOT_SMD:SOT-23-3, F.Cu at (166.8, 81.9)
- moved C12 3.25 mm to (227.2, 120.4), turned to 0 degrees
Connections:
- U1 pad 26: unconnected-(U1-PB0-Pad26) -> STM_Audio
- U3 pad 14: +5V -> Net-(B5819W-TP1-K)
Routing:
- net STM_Audio: track 0.00 -> 125.5 mm, vias 0 -> 4
- net Net-(B5819W-TP2-A): track 17.8 -> 30.9 mm
- net Net-(B5819W-TP1-K): track 0.00 -> 6.67 mm
- net +5V: track 125.9 -> 126.7 mm
- net GND: vias 129 -> 162

Commit message: 理想ダイオード変更前、一部修正
Parts:
- added C29: 0.1u, Capacitor_SMD:C_0603_1608Metric_Pad1.08x0.95mm_HandSolder, B.Cu at (186.7, 112.8)
Routing:
- net Net-(D6-A): track 3.51 -> 5.03 mm
Changed lines of the file:
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@@
 		)
 	)
+	(footprint "Capacitor_SMD:C_0603_1608Metric_Pad1.08x0.95mm_HandSolder"
+		(layer "B.Cu")
+		(at 186.7 112.8125 90)
+		(descr "Capacitor SMD 0603 (1608 Metric), square (rectangular) end terminal, IPC-7351 nominal with elongated pad for handsoldering. (Body size source: IPC-SM-782 page 76, https://www.pcb-3d.com/wordpress/wp-content/uploads/ipc-sm-782a_amendment_1_and_2.pdf)")
+		(tags "capacitor handsolder")
+		(property "Reference" "C29"
+			(at 0 1.43 90)
+			(layer "B.SilkS")
+			(hide yes)
+			(effects
+				(font
+					(size 1 1)
+					(thickness 0.15)
+				)
+				(justify mirror)
+			)
+		)
+		(property "Value" "0.1u"
+			(at 0 -1.43 90)
+			(layer "B.Fab")
+			(hide yes)
+			(effects
+				(font
+					(size 1 1)
+					(thickness 0.15)
+				)
+				(justify mirror)
+			)
+		)
+		(property "Datasheet" ""
+			(at 0 0 90)
+			(layer "B.Fab")
+			(hide yes)
+			(effects
+				(font
+					(size 1.27 1.27)
+				)
+				(justify mirror)
+			)
+		)
+		(property "Description" ""
+			(at 0 0 90)
+			(layer "B.Fab")
+			(hide yes)
+			(effects
+				(font
+					(size 1.27 1.27)
+				)
+				(justify mirror)
+			)
+		)
+		(property "KiLib_Generator" "SMD_2terminal_chip_molded"
+			(at 0 0 90)
+			(layer "B.SilkS")
+			(hide yes)
+			(effects
+				(font
+					(size 1 1)
+					(thickness 0.15)
+				)
+				(justify mirror)
+			)
+		)
+		(property ki_fp_filters "C_*")
+		(sheetname "/")
+		(sheetfile "MainBoard_V26_2_1.kicad_sch")
+		(units
+			(unit
+				(name "A")
+				(pins "1" "2")
+			)
+		)
+		(attr smd)
+		(duplicate_pad_numbers_are_jumpers no)
+		(fp_line
+			(start -0.146267 -0.51)
+			(end 0.146267 -0.51)
+			(stroke
+				(width 0.12)
+				(type solid)
+			)
+			(layer "B.SilkS")
+		)
+		(fp_line
+			(start -0.146267 0.51)
+			(end 0.146267 0.51)
+			(stroke
+				(width 0.12)
+				(type solid)
+			)
+			(layer "B.SilkS")
+		)
+		(fp_rect
+			(start -1.65 0.73)
+			(end 1.65 -0.73)
+			(stroke
+				(width 0.05)
+				(type solid)
+			)
+			(fill no)
+			(layer "B.CrtYd")
+		)
+		(fp_rect
+			(start -0.8 0.4)
+			(end 0.8 -0.4)
+			(stroke
+				(width 0.1)
+				(type solid)
+			)
+			(fill no)
+			(layer "B.Fab")
+		)
+		(fp_text user "${REFERENCE}"
+			(at 0 0 90)
+			(layer "B.Fab")
+			(effects
+				(font
+					(size 0.4 0.4)
+					(thickness 0.06)
+				)
+				(justify mirror)
+			)
+		)
+		(pad "1" smd roundrect
+			(at -0.8625 0 90)
+			(size 1.075 0.95)
+			(layers "B.Cu" "B.Mask" "B.Paste")
+			(roundrect_rratio 0.25)
+			(net "GND")
+			(pintype "passive")
+		)
+		(pad "2" smd roundrect
+			(at 0.8625 0 90)
+			(size 1.075 0.95)
+			(layers "B.Cu" "B.Mask" "B.Paste")
+			(roundrect_rratio 0.25)
+			(net "Net-(D6-A)")
+			(pintype "passive")
+		)
+		(embedded_fonts no)
+		(model "${KICAD10_3DMODEL_DIR}/Capacitor_SMD.3dshapes/C_0603_1608Metric.step"
+			(offset
+				(xyz 0 0 0)
+			)
+			(scale
+				(xyz 1 1 1)
+			)
+			(rotate
+				(xyz 0 0 0)
+			)
+		)
+	)
 	(gr_poly
 		(pts
@@
 	)
 	(segment
+		(start 186.667506 111.917506)
+		(end 186.7 111.95)
+		(width 0.2)
+		(layer "B.Cu")
+		(net "Net-(D6-A)")
+	)
+	(segment
 		(start 181.95 111.925)
 		(end 181.969994 111.905006)
@@
 		(width 0.2)
 		(layer "B.Cu")
+		(net "Net-(D6-A)")
+	)
+	(segment
+		(start 185.2 111.917506)
+		(end 186.667506 111.917506)
+		(width 0.2)
+		(layer "B.Cu")
