File: 2026/PCB/MainBoard/MainBoard_V26_2_1/MainBoard_V26_2_1.kicad_sch (KiCad schematic)
At the start: 93 parts, among them J1 Raspberry_Pi_2_3, J13 //Drib, J15 TFT3, J16 CAN_CON, J2 fan, J3 MOLEX, J5 Conn_01x05_Socket, J6 Debug, Q1 Q_NMOS_GSD, Q2 Q_NMOS_GSD, SW1 SW_MEC_5E, SW2 Ras_1, SW3 Ras_2, U1 STM32F446RETx, U2 LMR51460FSQDRRRQ1, U3 MOUDLE-SEEEDUINO-XIAO, U5 MCP1703AT-3302E/CB, U6 LSM6DSO32XTR, U7 LTC4451AV-TRPBF, U8 MAX3051, U9 LTC4451AV-TRPBF, Y1 CSTNE16M0V530000R0

Commit message: 途中保存
Parts:
- added Q3: Q_NMOS_GSD, Package_TO_SOT_SMD:SOT-23-3, symbol Device:Q_NMOS_GSD
- U4: value ~ -> (none)
Connections:
- net GND: now also Q3.2 (S)
- net at LS1.N, Q1.3 (D), Q2.3 (D)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: now also Q3.3 (D)
- new net STM_Audio: Q3.1 (G)

Commit message: 途中保存2
Parts:
- added B5819W-TP: D, symbol Device:D
Connections:
- net +5V: now also B5819W-TP.1 (K)
- net at LS1.N, Q1.3 (D), Q2.3 (D)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: now also B5819W-TP.2 (A)

Commit message: 修正完了。理想ダイオード変更前
Parts:
- added B5819W-TP1: D, Diode_SMD:D_SOD-123, symbol Device:D
- B5819W-TP2: renamed from B5819W-TP; footprint (none) -> Diode_SMD:D_SOD-123
Connections:
- net +5V: now also B5819W-TP1.2 (A); no longer U3.14 (5V)
- net STM_Audio: now also U1.26 (PB0)
- new net: B5819W-TP1.1 (K), U3.14 (5V)
- no-connect marks 35 -> 34
Changed lines of the file:
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@@
 	)
 	(junction
+		(at 316.23 212.09)
+		(diameter 0)
+		(color 0 0 0 0)
+	)
+	(junction
 		(at 127 38.1)
 		(diameter 0)
@@
 	)
 	(junction
-		(at 316.23 212.09)
-		(diameter 0)
-		(color 0 0 0 0)
-	)
-	(junction
 		(at 350.52 312.42)
 		(diameter 0)
@@
 	)
 	(no_connect
-		(at 135.89 107.95)
-	)
-	(no_connect
 		(at 129.54 320.04)
 	)
@@
 	(wire
 		(pts
+			(xy 316.23 212.09) (xy 316.23 217.17)
+		)
+		(stroke
+			(width 0)
+			(type default)
+		)
+	)
+	(wire
+		(pts
 			(xy 45.72 254) (xy 86.36 254)
 		)
@@
 	(wire
 		(pts
-			(xy 316.23 212.09) (xy 316.23 229.87)
-		)
-		(stroke
-			(width 0)
-			(type default)
-		)
-	)
-	(wire
-		(pts
 			(xy 482.6 198.12) (xy 482.6 199.39)
 		)
@@
 	(wire
 		(pts
+			(xy 316.23 224.79) (xy 316.23 229.87)
+		)
+		(stroke
+			(width 0)
+			(type default)
+		)
+	)
+	(wire
+		(pts
 			(xy 384.81 132.08) (xy 388.62 132.08)
 		)
@@
 	(global_label "STM_Audio"
 		(shape output)
-		(at 166.37 140.97 180)
+		(at 135.89 107.95 0)
 		(fields_autoplaced yes)
 		(effects
@@
 				(size 1.27 1.27)
 			)
-			(justify right)
+			(justify left)
 		)
 		(property "Intersheetrefs" "${INTERSHEET_REFS}"
-			(at 153.6483 140.97 0)
+			(at 148.6117 107.95 0)
 			(hide yes)
 			(show_name no)
@@
 					(size 1.27 1.27)
 				)
-				(justify right)
+				(justify left)
 			)
 		)
@@
 		(dnp no)
 		(fields_autoplaced yes)
-		(property "Reference" "B5819W-TP"
+		(property "Reference" "B5819W-TP2"
 			(at 434.34 40.6399 90)
 			(show_name no)
@@
 			)
 		)
-		(property "Footprint" ""
+		(property "Footprint" "Diode_SMD:D_SOD-123"
 			(at 431.8 41.91 0)
 			(hide yes)
@@
 			(project "MainBoard_V26_2_1"
 				(path "/1e41cf15-e032-452e-b093-2e98e4f5d157"
-					(reference "B5819W-TP")
+					(reference "B5819W-TP2")
 					(unit 1)
 				)
@@
 					(unit 1)
 				)
+			)
+		)
+	)
+	(symbol
+		(lib_id "Device:D")
+		(at 316.23 220.98 90)
+		(unit 1)
+		(body_style 1)
+		(exclude_from_sim no)
+		(in_bom yes)
+		(on_board yes)
+		(in_pos_files yes)
+		(dnp no)
+		(property "Reference" "B5819W-TP1"
+			(at 301.752 217.932 90)
+			(show_name no)
+			(do_not_autoplace no)
+			(effects
+				(font
+					(size 1.27 1.27)
+				)
+				(justify right)
+			)
+		)
+		(property "Value" "D"
+			(at 312.42 220.472 90)
+			(show_name no)
+			(do_not_autoplace no)
+			(effects
+				(font
+					(size 1.27 1.27)
+				)
+				(justify right)
+			)
+		)
+		(property "Footprint" "Diode_SMD:D_SOD-123"
+			(at 316.23 220.98 0)
+			(hide yes)
+			(show_name no)
+			(do_not_autoplace no)
+			(effects
+				(font
+					(size 1.27 1.27)
+				)
+			)
+		)
+		(property "Datasheet" ""
+			(at 316.23 220.98 0)
+			(hide yes)
+			(show_name no)
+			(do_not_autoplace no)
+			(effects
+				(font
+					(size 1.27 1.27)
+				)
+			)
+		)
+		(property "Description" "Diode"
+			(at 316.23 220.98 0)
+			(hide yes)
+			(show_name no)
+			(do_not_autoplace no)
+			(effects
+				(font
+					(size 1.27 1.27)
+				)
+			)
+		)
+		(property "Sim.Device" "D"
+			(at 316.23 220.98 0)
+			(hide yes)
+			(show_name no)
+			(do_not_autoplace no)
+			(effects
+				(font
+					(size 1.27 1.27)
+				)
+			)
+		)
+		(property "Sim.Pins" "1=K 2=A"
+			(at 316.23 220.98 0)
+			(hide yes)
+			(show_name no)
+			(do_not_autoplace no)
+			(effects
+				(font
+					(size 1.27 1.27)
+				)
+			)
+		)
+		(pin "2"
+		)
+		(pin "1"
+		)
+		(instances
+			(project "MainBoard_V26_2_1"
+				(path "/1e41cf15-e032-452e-b093-2e98e4f5d157"
+					(reference "B5819W-TP1")
+					(unit 1)
+				)

Commit message: 理想ダイオード変更前、一部修正
Parts:
- added C29: 0.1u, Capacitor_SMD:C_0603_1608Metric_Pad1.08x0.95mm_HandSolder, symbol Device:C
Connections:
- net GND: now also C29.1
- net at D6.2 (A), R10.2, R11.1: now also C29.2
Other:
- moved on the sheet: D6, R11
Changed lines of the file:
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@@
 	)
 	(junction
-		(at 306.07 59.69)
-		(diameter 0)
-		(color 0 0 0 0)
-	)
-	(junction
 		(at 215.9 295.91)
 		(diameter 0)
@@
 	)
 	(junction
+		(at 316.23 62.23)
+		(diameter 0)
+		(color 0 0 0 0)
+	)
+	(junction
 		(at 502.92 210.82)
 		(diameter 0)
@@
 	)
 	(junction
+		(at 306.07 62.23)
+		(diameter 0)
+		(color 0 0 0 0)
+	)
+	(junction
+		(at 306.07 78.74)
+		(diameter 0)
+		(color 0 0 0 0)
+	)
+	(junction
 		(at 271.78 143.51)
 		(diameter 0)
@@
 	(wire
 		(pts
-			(xy 306.07 68.58) (xy 306.07 74.93)
+			(xy 306.07 74.93) (xy 306.07 78.74)
 		)
 		(stroke
@@
 	(wire
 		(pts
+			(xy 306.07 57.15) (xy 306.07 62.23)
+		)
+		(stroke
+			(width 0)
+			(type default)
+		)
+	)
+	(wire
+		(pts
 			(xy 58.42 48.26) (xy 52.07 48.26)
 		)
@@
 		)
 	)
-	(polyline
+	(wire
 		(pts
-			(xy 80.01 128.27) (xy 80.01 97.79)
+			(xy 316.23 62.23) (xy 322.58 62.23)
 		)
 		(stroke
 			(width 0)
-			(type dash)
+			(type default)
 		)
 	)
-	(wire
+	(polyline
 		(pts
-			(xy 384.81 140.97) (xy 384.81 132.08)
+			(xy 80.01 128.27) (xy 80.01 97.79)
 		)
 		(stroke
 			(width 0)
-			(type default)
+			(type dash)
 		)
 	)
 	(wire
 		(pts
-			(xy 306.07 59.69) (xy 309.88 59.69)
+			(xy 384.81 140.97) (xy 384.81 132.08)
 		)
 		(stroke
@@
 	(wire
 		(pts
+			(xy 316.23 74.93) (xy 316.23 78.74)
+		)
+		(stroke
+			(width 0)
+			(type default)
+		)
+	)
+	(wire
+		(pts
 			(xy 473.71 198.12) (xy 473.71 199.39)
 		)
@@
 	(wire
 		(pts
+			(xy 306.07 62.23) (xy 306.07 67.31)
+		)
+		(stroke
+			(width 0)
+			(type default)
+		)
+	)
+	(wire
+		(pts
 			(xy 60.96 276.86) (xy 72.39 276.86)
 		)
@@
 	(wire
 		(pts
+			(xy 316.23 62.23) (xy 316.23 67.31)
+		)
+		(stroke
+			(width 0)
+			(type default)
+		)
+	)
+	(wire
+		(pts
 			(xy 74.93 36.83) (xy 74.93 38.1)
 		)
@@
 	(wire
 		(pts
-			(xy 306.07 59.69) (xy 306.07 60.96)
-		)
-		(stroke
-			(width 0)
-			(type default)
-		)
-	)
-	(wire
-		(pts
 			(xy 43.18 234.95) (xy 43.18 232.41)
 		)
@@
 	(wire
 		(pts
+			(xy 306.07 78.74) (xy 306.07 81.28)
+		)
+		(stroke
+			(width 0)
+			(type default)
+		)
+	)
+	(wire
+		(pts
 			(xy 502.92 187.96) (xy 502.92 190.5)
 		)
@@
 	(wire
 		(pts
-			(xy 306.07 57.15) (xy 306.07 59.69)
-		)
-		(stroke
-			(width 0)
-			(type default)
-		)
-	)
-	(wire
-		(pts
 			(xy 60.96 276.86) (xy 60.96 279.4)
 		)
@@
 	(wire
 		(pts
+			(xy 316.23 78.74) (xy 306.07 78.74)
+		)
+		(stroke
+			(width 0)
+			(type default)
+		)
+	)
+	(wire
+		(pts
 			(xy 422.91 82.55) (xy 422.91 88.9)
 		)
@@
 	(wire
 		(pts
-			(xy 317.5 59.69) (xy 320.04 59.69)
+			(xy 330.2 62.23) (xy 332.74 62.23)
 		)
 		(stroke
@@
 	(wire
 		(pts
+			(xy 306.07 62.23) (xy 316.23 62.23)
+		)
+		(stroke
+			(width 0)
+			(type default)
+		)
+	)
+	(wire
+		(pts
 			(xy 241.3 298.45) (xy 232.41 298.45)
 		)
@@
 	(global_label "BATTERY_MEASURE"
 		(shape input)
-		(at 320.04 59.69 0)
+		(at 332.74 62.23 0)
 		(fields_autoplaced yes)
 		(effects
@@
 		)
 		(property "Intersheetrefs" "${INTERSHEET_REFS}"
-			(at 340.4422 59.69 0)
+			(at 353.1422 62.23 0)
 			(hide yes)
 			(show_name no)
@@
 	(symbol
 		(lib_id "power:GND")
-		(at 306.07 74.93 0)
+		(at 306.07 81.28 0)
 		(unit 1)
 		(body_style 1)
@@
 		(dnp no)
 		(property "Reference" "#PWR032"
-			(at 306.07 81.28 0)
+			(at 306.07 87.63 0)
 			(hide yes)
 			(show_name no)
@@
 		)
 		(property "Value" "GND"
-			(at 306.07 80.01 0)
+			(at 306.07 86.36 0)
 			(show_name no)
 			(do_not_autoplace no)
@@
 		)
 		(property "Footprint" ""
-			(at 306.07 74.93 0)
+			(at 306.07 81.28 0)
 			(hide yes)
 			(show_name no)
@@
 		)
 		(property "Datasheet" ""
-			(at 306.07 74.93 0)
+			(at 306.07 81.28 0)
 			(hide yes)
 			(show_name no)
@@
 		)
 		(property "Description" ""
-			(at 306.07 74.93 0)
+			(at 306.07 81.28 0)
 			(show_name no)
 			(do_not_autoplace no)
@@
 	(symbol
 		(lib_id "Device:R")
-		(at 306.07 64.77 0)
+		(at 306.07 71.12 0)
 		(unit 1)
 		(body_style 1)
@@
 		(fields_autoplaced yes)
 		(property "Reference" "R11"
-			(at 308.61 63.4999 0)
+			(at 308.61 69.8499 0)
 			(show_name no)
 			(do_not_autoplace no)
@@
 		)
 		(property "Value" "10k"
-			(at 308.61 66.0399 0)
+			(at 308.61 72.3899 0)
 			(show_name no)
 			(do_not_autoplace no)
@@
 		)
 		(property "Footprint" "Resistor_SMD:R_0603_1608Metric_Pad0.98x0.95mm_HandSolder"
-			(at 304.292 64.77 90)
+			(at 304.292 71.12 90)
 			(hide yes)
 			(show_name no)
@@
 		)
 		(property "Datasheet" ""
-			(at 306.07 64.77 0)
+			(at 306.07 71.12 0)
 			(hide yes)
 			(show_name no)
@@
 		)
 		(property "Description" ""
-			(at 306.07 64.77 0)
+			(at 306.07 71.12 0)
 			(show_name no)
 			(do_not_autoplace no)
@@
 	(symbol
 		(lib_id "Diode:1N4148W")
-		(at 313.69 59.69 180)
+		(at 326.39 62.23 180)
 		(unit 1)
 		(body_style 1)
@@
 		(dnp no)
 		(property "Reference" "D6"
-			(at 317.5 62.23 0)
+			(at 330.2 64.77 0)
 			(show_name no)
 			(do_not_autoplace no)
@@
 		)
 		(property "Value" "1N4148W"
-			(at 317.5 64.77 0)
+			(at 330.2 67.31 0)
 			(show_name no)
 			(do_not_autoplace no)
@@
 		)
 		(property "Footprint" "Diode_SMD:D_SOD-123"
-			(at 313.69 55.245 0)
+			(at 326.39 57.785 0)
 			(hide yes)
 			(show_name no)
@@
 		)
 		(property "Datasheet" "https://www.vishay.com/docs/85748/1n4148w.pdf"
-			(at 313.69 59.69 0)
+			(at 326.39 62.23 0)
 			(hide yes)
 			(show_name no)
@@
 		)
 		(property "Description" ""
-			(at 313.69 59.69 0)
+			(at 326.39 62.23 0)
 			(show_name no)
 			(do_not_autoplace no)
@@
 		)
 		(property "Sim.Device" "D"
-			(at 313.69 59.69 0)
+			(at 326.39 62.23 0)
 			(hide yes)
 			(show_name no)
@@
 		)
 		(property "Sim.Pins" "1=K 2=A"
-			(at 313.69 59.69 0)
+			(at 326.39 62.23 0)
 			(hide yes)
 			(show_name no)
@@
 					(unit 1)
 				)
+			)
+		)
+	)
+	(symbol
+		(lib_id "Device:C")
+		(at 316.23 71.12 180)
+		(unit 1)
+		(body_style 1)
+		(exclude_from_sim no)
+		(in_bom yes)
+		(on_board yes)
+		(in_pos_files yes)
+		(dnp no)
+		(property "Reference" "C29"
+			(at 323.596 73.152 90)
+			(show_name no)
+			(do_not_autoplace no)
+			(effects
+				(font
+					(size 1.27 1.27)
+				)
+			)
+		)
+		(property "Value" "0.1u"
+			(at 321.056 73.152 90)
+			(show_name no)
+			(do_not_autoplace no)
+			(effects
+				(font
+					(size 1.27 1.27)
+				)
+			)
+		)
+		(property "Footprint" "Capacitor_SMD:C_0603_1608Metric_Pad1.08x0.95mm_HandSolder"
+			(at 315.2648 67.31 0)
+			(hide yes)
+			(show_name no)
+			(do_not_autoplace no)
+			(effects
+				(font
+					(size 1.27 1.27)
+				)
+			)
+		)
+		(property "Datasheet" ""
+			(at 316.23 71.12 0)
+			(hide yes)
+			(show_name no)
+			(do_not_autoplace no)
+			(effects
+				(font
+					(size 1.27 1.27)
+				)
+			)
+		)
+		(property "Description" ""
+			(at 316.23 71.12 0)
+			(show_name no)
+			(do_not_autoplace no)
+			(effects
+				(font
+					(size 1.27 1.27)
+				)
+			)
+		)
+		(pin "1"
+		)
+		(pin "2"
+		)
+		(instances
+			(project "MainBoard_V26_2_1"
+				(path "/1e41cf15-e032-452e-b093-2e98e4f5d157"
+					(reference "C29")
+					(unit 1)
+				)
